Commit message: working on 2wd

File: 2wd_robot_description/urdf/2wd_robot.xacro (robot description, xacro)
@@ -2,11 +2,12 @@
 <!-- THIS IS NECESSARY -->
 <robot name="2wd_robot" xmlns:xacro="http://www.ros.org/wiki/xacro">
-    <xacro:include filename="$(find mybot_description)/urdf/materials.xacro" />
-    <!--//////////////////////////// Moment of Interia Functions found in Wiki ////////////////////////////////// -->
-    <!-- Macro for calculating inertia of cylinder -->
+    <xacro:include filename="$(find 2wd_robot_description)/urdf/materials.xacro" /><!-- Include colors -->
+    <xacro:include filename="$(find 2wd_robot_description)/urdf/2wd_robot.gazebo" /><!-- Include Gazebo Tags -->
+    <!--//////////////////////////// Moment of Interia Functions ////////////////////////////////// -->
+    <!-- function for calculating inertia of cylinder -->
     <macro name="cylinder_inertia" params="m r h">
         <inertia ixx="${m*(3*r*r+h*h)/12}" ixy="0" ixz="0" iyx="0" iyy="${m*(3*r*r+h*h)/12}" iyz="0" izx="0" izy="0" izz="${m*r*r/2}" />
     </macro>
-    <!-- Macro for calculating inertia of cube -->
+    <!-- function for calculating inertia of cube -->
     <macro name="cube_inertia" params="w h d m">
         <inertia ixx="${m*(d*d+h*h)/12}" ixy="0" ixz="0" iyx="0" iyy="${m*(w*w+d*d)/12}" iyz="0" izx="0" izy="0" izz="${m*(w*w+h*h)/12}" />
@@ -25,5 +26,5 @@
         <inertial>
             <mass value="${base_mass}" />
-            <origin xyz="0 0 0" />
+            <origin xyz="0 0 0" rpy="${ninety_degrees} 0 0" />
             <cube_inertia m="${base_mass}" d="${base_depth}" h="${base_height}" w="${base_width}" />
         </inertial>
@@ -39,5 +40,5 @@
         <!-- 3) Add Collision for Base -->
         <collision>
-            <origin xyz="0 0 0" rpy="0 0 0 " />
+            <origin xyz="0 0 0" rpy="${ninety_degrees} 0 0 " />
             <geometry>
                 <!--length(depth) x width x height -->
@@ -49,5 +50,5 @@
           <origin xyz="-0.2 0 -0.125" rpy="0 0 0" />
           <geometry>
-            <sphere radius="0.08" />
+            <sphere radius="0.04" />
           </geometry>
         </visual>
@@ -56,5 +57,5 @@
           <origin xyz="-0.2 0 -0.125" rpy="0 0 0" />
           <geometry>
-            <sphere radius="0.08" />
+            <sphere radius="0.04" />
           </geometry>
         </collision>
@@ -77,5 +78,5 @@
             <origin xyz="0 0 0" rpy="0 0 0" /><!-- 90 because we want the wheel up not flat down -->
             <geometry>
-                <mesh filename="package://2wd_robot_description/meshes/wheel.stl" scale="1.25 1 1.25"/>
+                <mesh filename="package://2wd_robot_description/meshes/wheel.stl" scale="1 1 1"/>
             </geometry>
             <material name="grey" />
@@ -85,5 +86,5 @@
             <origin xyz="0 0 0" rpy="0 0 0 " />
             <geometry>
-                <mesh filename="package://2wd_robot_description/meshes/wheel.stl" scale="1.25 1 1.25"/>
+                <mesh filename="package://2wd_robot_description/meshes/wheel.stl" scale="1 1 1"/>
             </geometry>
         </collision>
@@ -101,5 +102,5 @@
             <origin xyz="0 0 0" rpy="0 0 0" /><!-- 90 because we want the wheel up not flat down -->
             <geometry>
-                <mesh filename="package://2wd_robot_description/meshes/wheel.stl" scale="1.25 1 1.25"/>
+                <mesh filename="package://2wd_robot_description/meshes/wheel.stl" scale="1 1 1"/>
             </geometry>
             <material name="grey" />
@@ -109,5 +110,5 @@
             <origin xyz="0 0 0" rpy="0 0 0 " />
             <geometry>
-                <mesh filename="package://2wd_robot_description/meshes/wheel.stl" scale="1.25 1 1.25"/>
+                <mesh filename="package://2wd_robot_description/meshes/wheel.stl" scale="1 1 1"/>
             </geometry>
         </collision>

Commit message: Added CPP files for motors

File: 2wd_robot_description/urdf/2wd_robot.xacro (robot description, xacro)
@@ -59,4 +59,17 @@
             <sphere radius="0.04" />
           </geometry>
+          <!-- Gazebo Physics -->
+          <surface>
+            <friction>
+                <ode>
+                    <!-- "mu" is the Coulomb friction coefficient for the first friction direction -->
+                    <mu> 0 </mu>
+                    <!-- "mu2" is the friction coefficient for the second friction direction (perpendicular to the first friction direction) -->
+                    <mu2> 0 </mu2>
+                    <slip1> 1.0 </slip1>
+                    <slip2> 1.0 </slip2>
+                </ode>
+            </friction>
+          </surface>
         </collision>
     </link>
@@ -130,4 +143,6 @@
         <!-- Axis of revoltuion. Right hand rule says Y will be rotating  -->
         <axis xyz="0 1 0" rpy="0 0 0" />
+        <!-- <limit> (required only for revolute and prismatic joint)  -->
+        <!-- <effort> An attribute for enforcing the maximum joint effort (|applied effort| < |effort|)  -->
     </joint>
     <!-- Left wheel <-> Base -->
